File: monRecti/untitled.brd (EAGLE design)
At the start: 93.3 x 87.5 mm, 69 parts, among them U1 PC817X2NIP0F, U10 PC817X2NIP0F, U2 PC817X2NIP0F, U3 PC817X2NIP0F, U4 PC817X2NIP0F, U5 PC817X2NIP0F, U6 PC817X2NIP0F, U7 PC817X2NIP0F, U8 PC817X2NIP0F, U9 PC817X2NIP0F, X1 MSTBA5, X2 MSTBA5, X3 MSTBA2, X4 MSTBA2, X7 MSTBA3, X8 MSTBA3

Commit message: revisi rangkaian
Parts:
- added ADS1: (no value), ds1115:ADS1115
- added X5, X6: MSTBA3, con-phoenix-508:MSTBA3
- moved X1 1.00 mm to (23.2, 1.88)
- moved X2 1.00 mm to (23.2, 85.6)
- moved X3 1.00 mm to (43.2, 1.87)
- moved X4 1.00 mm to (43.2, 85.6)
- moved X7 1.00 mm to (58.1, 1.90)
- moved X8 1.00 mm to (58.2, 85.6)
Connections:
- new net A0: ADS1.A0, X5.3
- new net A1: ADS1.A1, X5.2
- new net A2: ADS1.A2, X6.1
- new net A3: ADS1.A3, X6.2
- new net ADC0: TTGO1.4, X6.3
- new net ADC1: TTGO1.2, X5.1
- net GND: now also ADS1.ADDR, ADS1.GND
- net RX: now also TTGO1.16; no longer TTGO1.12
- net SCL: now also ADS1.SCL
- net SDA: now also ADS1.SDA
- net TX: now also TTGO1.17; no longer TTGO1.13
- net VCC: now also ADS1.VDD
Routing:
- net A1: track 0.00 -> 127.8 mm, vias 0 -> 1
- net A0: track 0.00 -> 113.1 mm, vias 0 -> 1
- net SCL: track 56.8 -> 124.4 mm, vias 0 -> 1
- net A3: track 0.00 -> 65.2 mm, vias 0 -> 1
- net A2: track 0.00 -> 65.1 mm, vias 0 -> 1
- net ADC1: track 0.00 -> 52.8 mm, vias 0 -> 2
- net SDA: track 123.2 -> 159.6 mm, vias 2 -> 3
- net ADC0: track 0.00 -> 26.2 mm
- net GND: track 276.3 -> 289.0 mm
- net RX: track 50.0 -> 62.2 mm
- net VCC: track 121.6 -> 128.9 mm
- net TX: track 50.2 -> 54.6 mm
- net TX1: track 76.7 -> 80.8 mm
- net RX1: track 65.5 -> 68.6 mm
- net COMM: track 274.2 -> 276.6 mm
Other:
- outline, holes or cut-outs redrawn
