File: monRecti/untitled.sch (EAGLE design)
At the start: 69 parts, among them U1 PC817X2NIP0F, U10 PC817X2NIP0F, U2 PC817X2NIP0F, U3 PC817X2NIP0F, U4 PC817X2NIP0F, U5 PC817X2NIP0F, U6 PC817X2NIP0F, U7 PC817X2NIP0F, U8 PC817X2NIP0F, U9 PC817X2NIP0F, X1 MSTBA5, X2 MSTBA5, X3 MSTBA2, X4 MSTBA2, X7 MSTBA3, X8 MSTBA3

Commit message: revisi rangkaian
Parts:
- added ADS1: (no value), ds1115:ADS1115
- added X5, X6: MSTBA3, con-phoenix-508:MSTBA3
Connections:
- new net A0: ADS1.A0, X5-3.1
- new net A1: ADS1.A1, X5-2.1
- new net A2: ADS1.A2, X6-1.1
- new net A3: ADS1.A3, X6-2.1
- new net ADC0: TTGO1.4, X6-3.1
- new net ADC1: TTGO1.2, X5-1.1
- net GND: now also ADS1.ADDR, ADS1.GND
- net RX: now also TTGO1.16; no longer TTGO1.12
- net SCL: now also ADS1.SCL
- net SDA: now also ADS1.SDA
- net TX: now also TTGO1.17; no longer TTGO1.13
- net VCC: now also ADS1.VDD
