File: monRectiv1.3/untitled.brd (EAGLE design)
At the start: 154 x 83.1 mm, 114 parts, among them IC1 MCP23017SS, J2 10118193-0001LF, Q1 12MHz, Q2 MMBT3904, Q3 MMBT3904, U1 PC817X2NIP0F, U10 PC817X2NIP0F, U11 ADS1115IDGSR, U12 CH340G, U13 ESP32-WROOM-32D, U14 AMS1117, U2 PC817X2NIP0F, U3 PC817X2NIP0F, U4 PC817X2NIP0F, U5 PC817X2NIP0F, U6 PC817X2NIP0F, U7 PC817X2NIP0F, U8 PC817X2NIP0F, U9 PC817X2NIP0F, X1 MSTBA5, X2 MSTBA5, X4 MSTBA4, X5 MSTBA3, X6 MSTBA3, X7 MSTBA2, X8 MSTBA2, X9 MSTBA3

Commit message: revisi PCBv1.3
Parts:
- added C11: 10uF, rcl:C0805K
- added C12: 100nF, rcl:C0805K
- added J1: U.FL-R-SMT(01), U.FL-R-SMT_01_:HRS_U.FL-R-SMT(01)
- added LORA-NICERF-V1: (no value), LORA-NICERF-V2:LORA-NICERF-V2
Connections:
- new net ANT: J1.3, LORA-NICERF-V1.ANT
- new net DIO0_LORA: LORA-NICERF-V1.DIO0, U13.10
- new net DIO1_LORA: LORA-NICERF-V1.DIO1, U13.11
- new net MISO_HSPI: LORA-NICERF-V1.MISO, U13.14
- new net MOSI_HSPI: LORA-NICERF-V1.MOSI, U13.16
- new net RST_LORA: LORA-NICERF-V1.NRST, U13.23
- new net SCK_HSPI: LORA-NICERF-V1.SCK, U13.13
- new net SS_LORA: LORA-NICERF-V1.NSS, U13.26
- net 3V3: now also C11.1, C12.1, LORA-NICERF-V1.VCC
- net GND: now also C11.2, C12.2, J1.1, J1.2, LORA-NICERF-V1.GND, LORA-NICERF-V1.GND1
Routing:
- net RST_LORA: track 0.00 -> 80.2 mm, vias 0 -> 2
- net SS_LORA: track 0.00 -> 71.4 mm, vias 0 -> 2
- net DIO0_LORA: track 0.00 -> 66.5 mm, vias 0 -> 2
- net SCK_HSPI: track 0.00 -> 65.9 mm, vias 0 -> 2
- net DIO1_LORA: track 0.00 -> 65.8 mm, vias 0 -> 2
- net MISO_HSPI: track 0.00 -> 64.8 mm, vias 0 -> 2
- net MOSI_HSPI: track 0.00 -> 58.3 mm, vias 0 -> 2
- net 3V3: track 189.7 -> 239.8 mm
- net GND: track 101.3 -> 110.5 mm, vias 34 -> 40
- net ANT: track 0.00 -> 4.48 mm
- net 12V: track 142.1 -> 141.1 mm
- net EN: track 65.2 -> 64.2 mm
Other:
- outline, holes or cut-outs redrawn
