File: monRectiv1.3/untitled.sch (EAGLE design)
At the start: 114 parts, among them IC1 MCP23017SS, J2 10118193-0001LF, Q1 12MHz, Q2 MMBT3904, Q3 MMBT3904, U1 PC817X2NIP0F, U10 PC817X2NIP0F, U11 ADS1115IDGSR, U12 CH340G, U13 ESP32-WROOM-32D, U14 AMS1117, U2 PC817X2NIP0F, U3 PC817X2NIP0F, U4 PC817X2NIP0F, U5 PC817X2NIP0F, U6 PC817X2NIP0F, U7 PC817X2NIP0F, U8 PC817X2NIP0F, U9 PC817X2NIP0F, X1 MSTBA5, X2 MSTBA5, X4 MSTBA4, X5 MSTBA3, X6 MSTBA3, X7 MSTBA2, X8 MSTBA2, X9 MSTBA3

Commit message: revisi PCBv1.3
Parts:
- added C11: 10uF, rcl:C-EUC0805K
- added C12: 100nF, rcl:C-EUC0805K
- added J1: U.FL-R-SMT(01), U.FL-R-SMT_01_:U.FL-R-SMT(01)
- added LORA-NICERF-V1: (no value), LORA-NICERF-V2:LORA-NICERF-V2
Connections:
- new net ANT: J1.SIG, LORA-NICERF-V1.ANT
- new net DIO0_LORA: LORA-NICERF-V1.DIO0, U13.IO25
- new net DIO1_LORA: LORA-NICERF-V1.DIO1, U13.IO26
- new net MISO_HSPI: LORA-NICERF-V1.MISO, U13.IO12
- new net MOSI_HSPI: LORA-NICERF-V1.MOSI, U13.IO13
- new net RST_LORA: LORA-NICERF-V1.NRST, U13.IO15
- new net SCK_HSPI: LORA-NICERF-V1.SCK, U13.IO14
- new net SS_LORA: LORA-NICERF-V1.NSS, U13.IO4
- net 3V3: now also C11.1, C12.1, LORA-NICERF-V1.VCC
- net GND: now also C11.2, C12.2, J1.GND, LORA-NICERF-V1.GND, LORA-NICERF-V1.GND1
Changed lines of the file:
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@@
 <part name="D13" library="SML-LXT0805IW-TR" deviceset="SML-LXT0805IW-TR" device=""/>
 <part name="GND15" library="supply1" library_urn="urn:adsk.eagle:library:371" deviceset="GND" device=""/>
+<part name="LORA-NICERF-V1" library="LORA-NICERF-V2" deviceset="LORA-NICERF-V2" device=""/>
+<part name="C11" library="rcl" library_urn="urn:adsk.eagle:library:334" deviceset="C-EU" device="C0805K" package3d_urn="urn:adsk.eagle:package:23681/2" value="10uF"/>
+<part name="C12" library="rcl" library_urn="urn:adsk.eagle:library:334" deviceset="C-EU" device="C0805K" package3d_urn="urn:adsk.eagle:package:23681/2" value="100nF"/>
+<part name="GND18" library="supply1" library_urn="urn:adsk.eagle:library:371" deviceset="GND" device=""/>
+<part name="GND19" library="supply1" library_urn="urn:adsk.eagle:library:371" deviceset="GND" device=""/>
+<part name="J1" library="U.FL-R-SMT_01_" deviceset="U.FL-R-SMT(01)" device=""/>
+<part name="GND20" library="supply1" library_urn="urn:adsk.eagle:library:371" deviceset="GND" device=""/>
 </parts>
 <sheets>
@@
 <instance part="GND15" gate="1" x="-114.3" y="-88.9" smashed="yes">
 <attribute name="VALUE" x="-116.84" y="-91.44" size="1.778" layer="96"/>
+</instance>
+<instance part="LORA-NICERF-V1" gate="G$1" x="66.04" y="-25.4" smashed="yes"/>
+<instance part="C11" gate="G$1" x="91.44" y="-27.94" smashed="yes">
+<attribute name="NAME" x="92.964" y="-27.559" size="1.778" layer="95"/>
+<attribute name="VALUE" x="92.964" y="-32.639" size="1.778" layer="96"/>
+</instance>
+<instance part="C12" gate="G$1" x="96.52" y="-27.94" smashed="yes">
+<attribute name="NAME" x="98.044" y="-27.559" size="1.778" layer="95"/>
+<attribute name="VALUE" x="98.044" y="-32.639" size="1.778" layer="96"/>
+</instance>
+<instance part="GND18" gate="1" x="35.56" y="-20.32" smashed="yes">
+<attribute name="VALUE" x="33.02" y="-22.86" size="1.778" layer="96"/>
+</instance>
+<instance part="GND19" gate="1" x="93.98" y="-35.56" smashed="yes">
+<attribute name="VALUE" x="91.44" y="-38.1" size="1.778" layer="96"/>
+</instance>
+<instance part="J1" gate="G$1" x="43.18" y="-43.18" smashed="yes">
+<attribute name="NAME" x="39.36143125" y="-39.10686875" size="1.27285" layer="95"/>
+<attribute name="VALUE" x="38.85218125" y="-48.7807" size="1.27288125" layer="96"/>
+</instance>
+<instance part="GND20" gate="1" x="30.48" y="-48.26" smashed="yes">
+<attribute name="VALUE" x="27.94" y="-50.8" size="1.778" layer="96"/>
 </instance>
 </instances>
@@
 <wire x1="-114.3" y1="-86.36" x2="-114.3" y2="-83.82" width="0.1524" layer="91"/>
 </segment>
+<segment>
+<pinref part="GND18" gate="1" pin="GND"/>
+<pinref part="LORA-NICERF-V1" gate="G$1" pin="GND"/>
+<wire x1="35.56" y1="-17.78" x2="50.8" y2="-17.78" width="0.1524" layer="91"/>
+<pinref part="LORA-NICERF-V1" gate="G$1" pin="GND1"/>
+<wire x1="78.74" y1="-20.32" x2="63.5" y2="-20.32" width="0.1524" layer="91"/>
+<wire x1="63.5" y1="-20.32" x2="63.5" y2="-17.78" width="0.1524" layer="91"/>
+<wire x1="63.5" y1="-17.78" x2="50.8" y2="-17.78" width="0.1524" layer="91"/>
+<junction x="50.8" y="-17.78"/>
+</segment>
+<segment>
+<pinref part="C11" gate="G$1" pin="2"/>
+<pinref part="C12" gate="G$1" pin="2"/>
+<wire x1="91.44" y1="-33.02" x2="93.98" y2="-33.02" width="0.1524" layer="91"/>
+<pinref part="GND19" gate="1" pin="GND"/>
+<wire x1="93.98" y1="-33.02" x2="96.52" y2="-33.02" width="0.1524" layer="91"/>
+<junction x="93.98" y="-33.02"/>
+</segment>
+<segment>
+<pinref part="GND20" gate="1" pin="GND"/>
+<pinref part="J1" gate="G$1" pin="GND"/>
+<wire x1="30.48" y1="-45.72" x2="33.02" y2="-45.72" width="0.1524" layer="91"/>
+</segment>
 </net>
 <net name="SDA" class="0">
@@
 <wire x1="-134.62" y1="-53.34" x2="-129.54" y2="-53.34" width="0.1524" layer="91"/>
 <label x="-132.08" y="-53.34" size="0.6096" layer="95" rot="R90" xref="yes"/>
+</segment>
+<segment>
+<pinref part="LORA-NICERF-V1" gate="G$1" pin="VCC"/>
+<pinref part="C11" gate="G$1" pin="1"/>
+<wire x1="78.74" y1="-25.4" x2="91.44" y2="-25.4" width="0.1524" layer="91"/>
+<pinref part="C12" gate="G$1" pin="1"/>
+<wire x1="91.44" y1="-25.4" x2="96.52" y2="-25.4" width="0.1524" layer="91"/>
+<junction x="91.44" y="-25.4"/>
+<wire x1="96.52" y1="-25.4" x2="99.06" y2="-25.4" width="0.1524" layer="91"/>
+<junction x="96.52" y="-25.4"/>
+<label x="99.06" y="-25.4" size="0.6096" layer="95" xref="yes"/>
 </segment>
 </net>
@@
 </segment>
 </net>
+<net name="SCK_HSPI" class="0">
+<segment>
+<pinref part="LORA-NICERF-V1" gate="G$1" pin="SCK"/>
+<wire x1="50.8" y1="-25.4" x2="48.26" y2="-25.4" width="0.1524" layer="91"/>
+<label x="48.26" y="-25.4" size="0.6096" layer="95" rot="R180" xref="yes"/>
+</segment>
+<segment>
+<pinref part="U13" gate="G$1" pin="IO14"/>
+<wire x1="91.44" y1="71.12" x2="93.98" y2="71.12" width="0.1524" layer="91"/>
+<label x="93.98" y="71.12" size="0.6096" layer="95" xref="yes"/>
+</segment>
+</net>
+<net name="MISO_HSPI" class="0">
+<segment>
+<pinref part="LORA-NICERF-V1" gate="G$1" pin="MISO"/>
+<wire x1="50.8" y1="-27.94" x2="48.26" y2="-27.94" width="0.1524" layer="91"/>
+<label x="48.26" y="-27.94" size="0.6096" layer="95" rot="R180" xref="yes"/>
+</segment>
+<segment>
+<pinref part="U13" gate="G$1" pin="IO12"/>
+<wire x1="91.44" y1="76.2" x2="93.98" y2="76.2" width="0.1524" layer="91"/>
+<label x="93.98" y="76.2" size="0.6096" layer="95" xref="yes"/>
+</segment>
+</net>
+<net name="MOSI_HSPI" class="0">
+<segment>
+<pinref part="LORA-NICERF-V1" gate="G$1" pin="MOSI"/>
+<wire x1="50.8" y1="-30.48" x2="48.26" y2="-30.48" width="0.1524" layer="91"/>
+<label x="48.26" y="-30.48" size="0.6096" layer="95" rot="R180" xref="yes"/>
+</segment>
+<segment>
+<pinref part="U13" gate="G$1" pin="IO13"/>
+<wire x1="91.44" y1="73.66" x2="93.98" y2="73.66" width="0.1524" layer="91"/>
+<label x="93.98" y="73.66" size="0.6096" layer="95" xref="yes"/>
+</segment>
+</net>
+<net name="SS_LORA" class="0">
+<segment>
+<pinref part="LORA-NICERF-V1" gate="G$1" pin="NSS"/>
+<wire x1="50.8" y1="-33.02" x2="48.26" y2="-33.02" width="0.1524" layer="91"/>
+<label x="48.26" y="-33.02" size="0.6096" layer="95" rot="R180" xref="yes"/>
+</segment>
+<segment>
+<pinref part="U13" gate="G$1" pin="IO4"/>
+<wire x1="91.44" y1="81.28" x2="93.98" y2="81.28" width="0.1524" layer="91"/>
+<label x="93.98" y="81.28" size="0.6096" layer="95" xref="yes"/>
+</segment>
+</net>
+<net name="ANT" class="0">
+<segment>
+<pinref part="LORA-NICERF-V1" gate="G$1" pin="ANT"/>
+<wire x1="78.74" y1="-17.78" x2="81.28" y2="-17.78" width="0.1524" layer="91"/>
+<label x="81.28" y="-17.78" size="0.6096" layer="95" xref="yes"/>
+</segment>
+<segment>
+<pinref part="J1" gate="G$1" pin="SIG"/>
+<wire x1="33.02" y1="-40.64" x2="30.48" y2="-40.64" width="0.1524" layer="91"/>
+<label x="30.48" y="-40.64" size="0.6096" layer="95" rot="R180" xref="yes"/>
+</segment>
+</net>
+<net name="RST_LORA" class="0">
+<segment>
+<pinref part="LORA-NICERF-V1" gate="G$1" pin="NRST"/>
+<wire x1="78.74" y1="-22.86" x2="81.28" y2="-22.86" width="0.1524" layer="91"/>
+<label x="81.28" y="-22.86" size="0.6096" layer="95" xref="yes"/>
+</segment>
+<segment>
+<pinref part="U13" gate="G$1" pin="IO15"/>
+<wire x1="93.98" y1="68.58" x2="91.44" y2="68.58" width="0.1524" layer="91"/>
+<label x="93.98" y="68.58" size="0.6096" layer="95" xref="yes"/>
+</segment>
+</net>
+<net name="DIO0_LORA" class="0">
+<segment>
+<pinref part="LORA-NICERF-V1" gate="G$1" pin="DIO0"/>
+<wire x1="78.74" y1="-27.94" x2="81.28" y2="-27.94" width="0.1524" layer="91"/>
+<label x="81.28" y="-27.94" size="0.6096" layer="95" xref="yes"/>
+</segment>
+<segment>
+<pinref part="U13" gate="G$1" pin="IO25"/>
+<wire x1="91.44" y1="48.26" x2="93.98" y2="48.26" width="0.1524" layer="91"/>
+<label x="93.98" y="48.26" size="0.6096" layer="95" xref="yes"/>
+</segment>
+</net>
+<net name="DIO1_LORA" class="0">
+<segment>
+<pinref part="LORA-NICERF-V1" gate="G$1" pin="DIO1"/>
+<wire x1="78.74" y1="-30.48" x2="81.28" y2="-30.48" width="0.1524" layer="91"/>
+<label x="81.28" y="-30.48" size="0.6096" layer="95" xref="yes"/>
+</segment>
+<segment>
+<pinref part="U13" gate="G$1" pin="IO26"/>
+<wire x1="91.44" y1="45.72" x2="93.98" y2="45.72" width="0.1524" layer="91"/>
+<label x="93.98" y="45.72" size="0.6096" layer="95" xref="yes"/>
+</segment>
+</net>
